File: type5.kicad_pcb (KiCad board)
At the start: 2 copper layers, 80 x 50 mm, 3 parts, among them P1 CONN_01X09, P2 CONN_01X26, U1 TEENSYPP2

Commit message: pcb mod
Parts:
- U1: moved to B.Cu
- moved P2 48.0 mm to (153.8, 120.0)
- moved P1 46.9 mm to (113.8, 121.2)
- moved U1 7.59 mm to (145.4, 96.1)
Routing:
- net Net-(P1-Pad2): track 71.5 -> 93.1 mm
- net Net-(P1-Pad1): track 77.4 -> 97.1 mm
- net Net-(P2-Pad26): track 75.4 -> 91.9 mm
- net Net-(P1-Pad4): track 63.8 -> 79.9 mm
- net Net-(P2-Pad24): track 67.6 -> 82.3 mm
- net Net-(P1-Pad3): track 69.6 -> 84.0 mm
- net Net-(P2-Pad22): track 59.8 -> 72.7 mm
- net Net-(P2-Pad20): track 51.3 -> 63.1 mm
- net Net-(P2-Pad25): track 73.5 -> 84.6 mm
- net Net-(P1-Pad6): track 56.0 -> 66.8 mm
- net Net-(P2-Pad1): track 34.5 -> 23.9 mm
- net Net-(P2-Pad5): track 31.9 -> 21.8 mm
- net Net-(P2-Pad3): track 32.6 -> 22.8 mm
- net Net-(P2-Pad23): track 65.7 -> 75.0 mm
- net Net-(P2-Pad16): track 17.1 -> 26.2 mm
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Other:
- board size 80 x 50 mm -> 87.5 x 66.2 mm

Commit message: pcb mod and drill
Parts:
- P1, P2: moved to B.Cu
- U1: moved to F.Cu
- moved P1 50.1 mm to (111.2, 71.2)
- moved P2 47.6 mm to (151.2, 72.5)
- moved U1 2.53 mm to (142.9, 96.6)
Other:
- outline, holes or cut-outs redrawn

Commit message: mod
Parts:
- moved P1 1.25 mm to (110.0, 71.2)
- moved P2 1.25 mm to (150.0, 72.5)
- moved U1 0.46 mm to (142.9, 96.1)
Connections:
- U1 pad 1: Net-(U1-Pad1) -> Net-(P2-Pad4)
- U1 pad 47: Net-(P2-Pad4) -> Net-(U1-Pad47)
Routing:
- net Net-(P2-Pad4): track 24.8 -> 54.5 mm
- net Net-(P1-Pad1): track 97.1 -> 83.7 mm
- net Net-(P1-Pad2): track 93.1 -> 81.4 mm
- net Net-(P1-Pad3): track 84.0 -> 74.1 mm
- net Net-(P1-Pad4): track 79.9 -> 71.8 mm
- net Net-(P1-Pad5): track 70.8 -> 64.5 mm
- net Net-(P1-Pad6): track 66.8 -> 62.2 mm
- net Net-(P1-Pad7): track 57.7 -> 54.9 mm
- net Net-(P1-Pad8): track 53.6 -> 52.6 mm
- net Net-(P2-Pad22): track 72.7 -> 73.5 mm
- net Net-(P2-Pad21): track 65.4 -> 66.2 mm
- net Net-(P2-Pad20): track 63.1 -> 63.8 mm
- net Net-(P2-Pad17): track 46.2 -> 46.9 mm
- net Net-(P2-Pad25): track 84.6 -> 85.4 mm
- net Net-(P2-Pad24): track 82.3 -> 83.0 mm
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Other:
- board size 87.5 x 66.2 mm -> 83.8 x 57.5 mm

Commit message: adsù
Other:
- net class Default: clearance 0.25 -> 0.1; trace_width 0.25 -> 0.35
- rule trace_clearance: 0.25 -> 0.1

Commit message: fix
Connections:
- U1 pad 1: Net-(P2-Pad4) -> Net-(P2-Pad23)
- U1 pad 14: Net-(P2-Pad23) -> Net-(U1-Pad14)
- U1 pad 47: Net-(U1-Pad47) -> Net-(P2-Pad4)
Routing:
- net Net-(P2-Pad4): track 54.5 -> 24.0 mm
- net Net-(P2-Pad23): track 75.7 -> 81.5 mm
