File: type5.kicad_pcb (KiCad board)
At the start: 2 copper layers, 85 x 70 mm, 3 parts, among them P1 CONN_01X09, P2 CONN_01X26, U1 TEENSYPP2

Commit message: finish (hope)
Parts:
- added R1: R, Resistors_ThroughHole:Resistor_Horizontal_RM7mm, F.Cu at (131.2, 82.6)
Connections:
- U1 pad 1: Net-(P2-Pad23) -> Net-(U1-Pad1)
Routing:
- net Net-(P2-Pad23): track 92.4 -> 47.4 mm
- net Net-(R1-Pad1): track 0.00 -> 19.3 mm
Other:
- board text added: "Dev in CrunchLab"
- board text added: "Made in LinoLab"
