File: type5.sch (KiCad schematic (older format))
At the start: 3 parts, among them P1 CONN_01X09, P2 CONN_01X26, U1 TEENSYPP2

Commit message: fix
Connections:
- net at U1.1 (GND): now also P2.23 (P23); no longer P2.4 (P4)
- net at U1.14 (PC1): no longer P2.23 (P23)
- net at U1.47 (PB2): now also P2.4 (P4)
- no-connect marks 18 -> 19
Changed lines of the file:
@@
 	3850 5500 3850 6050
-Wire Wire Line
-	3750 6050 3750 5550
-Wire Wire Line
-	3750 5550 2850 5550
-Wire Wire Line
-	2850 5550 2850 4000
-Wire Wire Line
-	2850 4000 3150 4000
 Wire Wire Line
 	3150 3900 2800 3900
@@
 	2300 3600 3150 3600
 Wire Wire Line
-	5650 6650 5650 6050
+	1650 2700 3150 2700
 Wire Wire Line
-	1650 6650 5650 6650
+	5650 6050 5650 5750
 Wire Wire Line
-	1650 6650 1650 2700
+	5650 5750 6500 5750
 Wire Wire Line
-	1650 2700 3150 2700
+	6500 5750 6500 3200
+Wire Wire Line
+	6500 3200 5850 3200
+Wire Wire Line
+	3750 6050 3750 6400
+Wire Wire Line
+	3750 6400 1650 6400
+Wire Wire Line
+	1650 6400 1650 2700
+NoConn ~ 3150 4000
 $EndSCHEMATC
